File: macropad.kicad_pcb (KiCad board)
At the start: 2 copper layers, 66 x 45.7 mm, 14 parts, among them J1 Conn_01x03_Pin, J2 Conn_01x02_Pin, SW1 SW_Push, SW2 SW_Push, SW3 SW_Push, U1 XIAO-RP2040-DIP

Commit message: Rewire power LED to 3V
Connections:
- U1 pad 12: unconnected-(U1-3V3-Pad12)_1 -> Power
- U1 pad 14: Power -> unconnected-(U1-VBUS-Pad14)_1
Routing:
- net Power: track 51.6 -> 45.3 mm, vias 0 -> 1
Changed lines of the file:
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@@
 	(net 9 "S2")
 	(net 10 "S3")
-	(net 11 "unconnected-(U1-3V3-Pad12)")
+	(net 11 "unconnected-(U1-VBUS-Pad14)")
 	(net 12 "unconnected-(U1-GPIO1{slash}RX-Pad8)")
 	(net 13 "unconnected-(U1-GPIO0{slash}TX-Pad7)")
@@
 	(net 17 "IO2")
 	(net 18 "Power")
-	(net 19 "unconnected-(U1-3V3-Pad12)_1")
+	(net 19 "unconnected-(U1-VBUS-Pad14)_1")
 	(net 20 "unconnected-(U1-GPIO1{slash}RX-Pad8)_1")
 	(net 21 "unconnected-(U1-GPIO0{slash}TX-Pad7)_1")
@@
 			(layers "*.Cu" "*.Mask")
 			(remove_unused_layers no)
-			(net 11 "unconnected-(U1-3V3-Pad12)")
+			(net 18 "Power")
 			(pinfunction "3V3")
-			(pintype "passive+no_connect")
+			(pintype "passive")
 		)
 		(pad "12" smd roundrect
@@
 			(layers "F.Cu" "F.Mask")
 			(roundrect_rratio 0.1)
-			(net 19 "unconnected-(U1-3V3-Pad12)_1")
+			(net 18 "Power")
 			(pinfunction "3V3")
-			(pintype "passive+no_connect")
+			(pintype "passive")
 			(thermal_bridge_angle 45)
 		)
@@
 			(layers "*.Cu" "*.Mask")
 			(remove_unused_layers no)
-			(net 18 "Power")
+			(net 11 "unconnected-(U1-VBUS-Pad14)")
 			(pinfunction "VBUS")
-			(pintype "passive")
+			(pintype "passive+no_connect")
 		)
 		(pad "14" smd roundrect
@@
 			(layers "F.Cu" "F.Mask")
 			(roundrect_rratio 0.1)
-			(net 18 "Power")
+			(net 19 "unconnected-(U1-VBUS-Pad14)_1")
 			(pinfunction "VBUS")
-			(pintype "passive")
+			(pintype "passive+no_connect")
 			(thermal_bridge_angle 45)
 		)
@@
 	)
 	(segment
-		(start 155.7635 78.2935)
-		(end 155.7635 70.6735)
-		(width 0.2)
-		(layer "F.Cu")
-		(net 18)
-	)
-	(segment
 		(start 152.908 86.36)
 		(end 150.109 86.36)
@@
 	)
 	(segment
-		(start 155.194 70.104)
-		(end 125.295 70.104)
+		(start 131.826 75.184)
+		(end 132.08 75.438)
 		(width 0.2)
 		(layer "F.Cu")
@@
 	)
 	(segment
-		(start 155.7635 70.6735)
-		(end 155.194 70.104)
+		(start 125.295 75.184)
+		(end 131.826 75.184)
 		(width 0.2)
 		(layer "F.Cu")
@@
 	)
 	(segment
-		(start 155.7635 78.2935)
-		(end 155.317 78.74)
+		(start 132.08 75.438)
+		(end 132.08 76.708)
 		(width 0.2)
 		(layer "F.Cu")
 		(net 18)
 	)
+	(via
+		(at 132.08 76.708)
+		(size 0.6)
+		(drill 0.3)
+		(layers "F.Cu" "B.Cu")
+		(net 18)
+	)
 	(segment
-		(start 155.317 78.74)
+		(start 132.08 76.708)
+		(end 132.08 80.264)
+		(width 0.2)
+		(layer "B.Cu")
+		(net 18)
+	)
+	(segment
+		(start 153.162 80.264)
 		(end 153.162 78.74)
 		(width 0.2)
-		(layer "F.Cu")
+		(layer "B.Cu")
+		(net 18)
+	)
+	(segment
+		(start 132.08 80.264)
+		(end 132.588 80.772)
+		(width 0.2)
+		(layer "B.Cu")
+		(net 18)
+	)
+	(segment
+		(start 152.654 80.772)
+		(end 153.162 80.264)
+		(width 0.2)
+		(layer "B.Cu")
+		(net 18)
+	)
+	(segment
+		(start 132.588 80.772)
+		(end 152.654 80.772)
+		(width 0.2)
+		(layer "B.Cu")
 		(net 18)
 	)
