File: macro-microcontroller.kicad_pcb (KiCad board)
At the start: 2 copper layers, 66 x 45.7 mm, 15 parts, among them J1 Conn_01x03_Pin, J2 Conn_01x02_Pin, SW1 SW_Push, SW2 SW_Push, SW3 SW_Push, U1 XIAO-RP2040-DIP

Commit message: Minor edits to firmware and schematic
Connections:
- net S1 renamed SW1
- net S2 renamed SW2
- net S3 renamed SW3
Changed lines of the file:
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@@
 	(net 6 "LED2")
 	(net 7 "LED3")
-	(net 8 "S1")
-	(net 9 "S2")
-	(net 10 "S3")
+	(net 8 "SW1")
+	(net 9 "SW2")
+	(net 10 "SW3")
 	(net 11 "+5V")
 	(net 12 "unconnected-(U1-GPIO1{slash}RX-Pad8)")
@@
 		)
 		(sheetname "/")
-		(sheetfile "macropad.kicad_sch")
+		(sheetfile "macro-microcontroller.kicad_sch")
 		(attr through_hole)
 		(fp_line
@@
 		)
 		(sheetname "/")
-		(sheetfile "macropad.kicad_sch")
+		(sheetfile "macro-microcontroller.kicad_sch")
 		(attr smd)
 		(fp_line
@@
 			(layers "F.Cu" "F.Mask")
 			(roundrect_rratio 0.1)
-			(net 8 "S1")
+			(net 8 "SW1")
 			(pinfunction "GPIO29/ADC3/A3")
 			(pintype "passive")
@@
 			(layers "*.Cu" "*.Mask")
 			(remove_unused_layers no)
-			(net 8 "S1")
+			(net 8 "SW1")
 			(pinfunction "GPIO29/ADC3/A3")
 			(pintype "passive")
@@
 			(layers "F.Cu" "F.Mask")
 			(roundrect_rratio 0.1)
-			(net 9 "S2")
+			(net 9 "SW2")
 			(pinfunction "GPIO6/SDA")
 			(pintype "passive")
@@
 			(layers "*.Cu" "*.Mask")
 			(remove_unused_layers no)
-			(net 9 "S2")
+			(net 9 "SW2")
 			(pinfunction "GPIO6/SDA")
 			(pintype "passive")
@@
 			(layers "F.Cu" "F.Mask")
 			(roundrect_rratio 0.1)
-			(net 10 "S3")
+			(net 10 "SW3")
 			(pinfunction "GPIO7/SCL")
 			(pintype "passive")
@@
 			(layers "*.Cu" "*.Mask")
 			(remove_unused_layers no)
-			(net 10 "S3")
+			(net 10 "SW3")
 			(pinfunction "GPIO7/SCL")
 			(pintype "passive")
@@
 		(property ki_fp_filters "R_*")
 		(sheetname "/")
-		(sheetfile "macropad.kicad_sch")
+		(sheetfile "macro-microcontroller.kicad_sch")
 		(attr through_hole)
 		(fp_line
@@
 		(property ki_fp_filters "R_*")
 		(sheetname "/")
-		(sheetfile "macropad.kicad_sch")
+		(sheetfile "macro-microcontroller.kicad_sch")
 		(attr through_hole)
 		(fp_line
@@
 		)
 		(sheetname "/")
-		(sheetfile "macropad.kicad_sch")
+		(sheetfile "macro-microcontroller.kicad_sch")
 		(attr through_hole)
 		(fp_line
@@
 			(layers "*.Cu" "*.Mask")
 			(remove_unused_layers no)
-			(net 10 "S3")
+			(net 10 "SW3")
 			(pinfunction "1")
 			(pintype "passive")
@@
 		)
 		(sheetname "/")
-		(sheetfile "macropad.kicad_sch")
+		(sheetfile "macro-microcontroller.kicad_sch")
 		(attr through_hole)
 		(fp_line
@@
 		(property ki_fp_filters "Connector*:*_1x??_*")
 		(sheetname "/")
-		(sheetfile "macropad.kicad_sch")
+		(sheetfile "macro-microcontroller.kicad_sch")
 		(attr through_hole)
 		(fp_line
@@
 		(property ki_fp_filters "Connector*:*_1x??_*")
 		(sheetname "/")
-		(sheetfile "macropad.kicad_sch")
+		(sheetfile "macro-microcontroller.kicad_sch")
 		(attr through_hole)
 		(fp_line
@@
 		(property ki_fp_filters "R_*")
 		(sheetname "/")
-		(sheetfile "macropad.kicad_sch")
+		(sheetfile "macro-microcontroller.kicad_sch")
 		(attr through_hole)
 		(fp_line
@@
 		)
 		(sheetname "/")
-		(sheetfile "macropad.kicad_sch")
+		(sheetfile "macro-microcontroller.kicad_sch")
 		(attr through_hole)
 		(fp_line
@@
 		)
 		(sheetname "/")
-		(sheetfile "macropad.kicad_sch")
+		(sheetfile "macro-microcontroller.kicad_sch")
 		(attr through_hole)
 		(fp_line
@@
 		(property ki_fp_filters "R_*")
 		(sheetname "/")
-		(sheetfile "macropad.kicad_sch")
+		(sheetfile "macro-microcontroller.kicad_sch")
 		(attr through_hole)
 		(fp_line
@@
 		)
 		(sheetname "/")
-		(sheetfile "macropad.kicad_sch")
+		(sheetfile "macro-microcontroller.kicad_sch")
 		(attr through_hole)
 		(fp_line
@@
 			(layers "*.Cu" "*.Mask")
 			(remove_unused_layers no)
-			(net 9 "S2")
+			(net 9 "SW2")
 			(pinfunction "1")
 			(pintype "passive")
@@
 		)
 		(sheetname "/")
-		(sheetfile "macropad.kicad_sch")
+		(sheetfile "macro-microcontroller.kicad_sch")
 		(attr through_hole)
 		(fp_line
@@
 			(layers "*.Cu" "*.Mask")
 			(remove_unused_layers no)
-			(net 8 "S1")
+			(net 8 "SW1")
 			(pinfunction "1")
 			(pintype "passive")
@@
 		(property ki_fp_filters "Potentiometer*")
 		(sheetname "/")
-		(sheetfile "macropad.kicad_sch")
+		(sheetfile "macro-microcontroller.kicad_sch")
 		(attr through_hole)
 		(fp_line
