File: macro-microcontroller.kicad_sch (KiCad schematic)
At the start: 15 parts, among them J1 Conn_01x03_Pin, J2 Conn_01x02_Pin, SW1 SW_Push, SW2 SW_Push, SW3 SW_Push, U1 XIAO-RP2040-DIP

Commit message: Minor edits to firmware and schematic
Connections:
- net S1 renamed SW1
- net S2 renamed SW2
- net S3 renamed SW3
Other:
- moved on the sheet: SW2, SW3
Changed lines of the file:
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@@
 		(at 153.67 101.6)
 	)
-	(global_label "S1"
+	(global_label "SW1"
 		(shape input)
 		(at 90.17 53.34 180)
@@
 		)
 		(property "Intersheetrefs" "${INTERSHEET_REFS}"
-			(at 84.7658 53.34 0)
+			(at 83.3144 53.34 0)
 			(effects
 				(font
@@
 		)
 	)
-	(global_label "S2"
+	(global_label "SW2"
 		(shape input)
 		(at 118.11 93.98 180)
@@
 		)
 		(property "Intersheetrefs" "${INTERSHEET_REFS}"
-			(at 112.7058 93.98 0)
+			(at 111.2544 93.98 0)
 			(effects
 				(font
@@
 		)
 	)
-	(global_label "S1"
+	(global_label "SW1"
 		(shape input)
 		(at 118.11 90.17 180)
@@
 		)
 		(property "Intersheetrefs" "${INTERSHEET_REFS}"
-			(at 112.7058 90.17 0)
+			(at 111.2544 90.17 0)
 			(effects
 				(font
@@
 		)
 	)
-	(global_label "S3"
+	(global_label "SW3"
 		(shape input)
-		(at 125.73 53.34 180)
+		(at 128.27 53.34 180)
 		(fields_autoplaced yes)
 		(effects
@@
 		)
 		(property "Intersheetrefs" "${INTERSHEET_REFS}"
-			(at 120.3258 53.34 0)
+			(at 121.4144 53.34 0)
 			(effects
 				(font
@@
 		)
 	)
-	(global_label "S2"
+	(global_label "SW2"
 		(shape input)
-		(at 107.95 53.34 180)
+		(at 109.22 53.34 180)
 		(fields_autoplaced yes)
 		(effects
@@
 		)
 		(property "Intersheetrefs" "${INTERSHEET_REFS}"
-			(at 102.5458 53.34 0)
+			(at 102.3644 53.34 0)
 			(effects
 				(font
@@
 		)
 	)
-	(global_label "S3"
+	(global_label "SW3"
 		(shape input)
 		(at 118.11 97.79 180)
@@
 		)
 		(property "Intersheetrefs" "${INTERSHEET_REFS}"
-			(at 112.7058 97.79 0)
+			(at 111.2544 97.79 0)
 			(effects
 				(font
@@
 	(symbol
 		(lib_id "Switch:SW_Push")
-		(at 130.81 53.34 0)
+		(at 133.35 53.34 0)
 		(unit 1)
 		(exclude_from_sim no)
@@
 		(fields_autoplaced yes)
 		(property "Reference" "SW3"
-			(at 130.81 45.72 0)
+			(at 133.35 45.72 0)
 			(effects
 				(font
@@
 		)
 		(property "Value" "SW_Push"
-			(at 130.81 48.26 0)
+			(at 133.35 48.26 0)
 			(effects
 				(font
@@
 		)
 		(property "Footprint" "Button_Switch_Keyboard:SW_Cherry_MX_1.00u_PCB"
-			(at 130.81 48.26 0)
+			(at 133.35 48.26 0)
 			(effects
 				(font
@@
 		)
 		(property "Datasheet" "~"
-			(at 130.81 48.26 0)
+			(at 133.35 48.26 0)
 			(effects
 				(font
@@
 		)
 		(property "Description" "Push button switch, generic, two pins"
-			(at 130.81 53.34 0)
+			(at 133.35 53.34 0)
 			(effects
 				(font
@@
 	(symbol
 		(lib_id "power:GND")
-		(at 118.11 53.34 0)
+		(at 119.38 53.34 0)
 		(unit 1)
 		(exclude_from_sim no)
@@
 		(fields_autoplaced yes)
 		(property "Reference" "#PWR02"
-			(at 118.11 59.69 0)
+			(at 119.38 59.69 0)
 			(effects
 				(font
@@
 		)
 		(property "Value" "GND"
-			(at 118.11 58.42 0)
+			(at 119.38 58.42 0)
 			(effects
 				(font
@@
 		)
 		(property "Footprint" ""
-			(at 118.11 53.34 0)
+			(at 119.38 53.34 0)
 			(effects
 				(font
@@
 		)
 		(property "Datasheet" ""
-			(at 118.11 53.34 0)
+			(at 119.38 53.34 0)
 			(effects
 				(font
@@
 		)
 		(property "Description" "Power symbol creates a global label with name \"GND\" , ground"
-			(at 118.11 53.34 0)
+			(at 119.38 53.34 0)
 			(effects
 				(font
@@
 	(symbol
 		(lib_id "power:GND")
-		(at 135.89 53.34 0)
+		(at 138.43 53.34 0)
 		(unit 1)
 		(exclude_from_sim no)
@@
 		(fields_autoplaced yes)
 		(property "Reference" "#PWR03"
-			(at 135.89 59.69 0)
+			(at 138.43 59.69 0)
 			(effects
 				(font
@@
 		)
 		(property "Value" "GND"
-			(at 135.89 58.42 0)
+			(at 138.43 58.42 0)
 			(effects
 				(font
@@
 		)
 		(property "Footprint" ""
-			(at 135.89 53.34 0)
+			(at 138.43 53.34 0)
 			(effects
 				(font
@@
 		)
 		(property "Datasheet" ""
-			(at 135.89 53.34 0)
+			(at 138.43 53.34 0)
 			(effects
 				(font
@@
 		)
 		(property "Description" "Power symbol creates a global label with name \"GND\" , ground"
-			(at 135.89 53.34 0)
+			(at 138.43 53.34 0)
 			(effects
 				(font
@@
 	(symbol
 		(lib_id "Switch:SW_Push")
-		(at 113.03 53.34 0)
+		(at 114.3 53.34 0)
 		(unit 1)
 		(exclude_from_sim no)
@@
 		(fields_autoplaced yes)
 		(property "Reference" "SW2"
-			(at 113.03 45.72 0)
+			(at 114.3 45.72 0)
 			(effects
 				(font
@@
 		)
 		(property "Value" "SW_Push"
-			(at 113.03 48.26 0)
+			(at 114.3 48.26 0)
 			(effects
 				(font
@@
 		)
 		(property "Footprint" "Button_Switch_Keyboard:SW_Cherry_MX_1.00u_PCB"
-			(at 113.03 48.26 0)
+			(at 114.3 48.26 0)
 			(effects
 				(font
@@
 		)
 		(property "Datasheet" "~"
-			(at 113.03 48.26 0)
+			(at 114.3 48.26 0)
 			(effects
 				(font
@@
 		)
 		(property "Description" "Push button switch, generic, two pins"
-			(at 113.03 53.34 0)
-			(effects
-				(font
+			(at 114.3 53.34 0)
+			(effects
+				(font
